File: kicad/prog-cc-100mA.kicad_pcb (KiCad board)
At the start: 2 copper layers, 49.5 x 49.5 mm, 39 parts, among them IC1 ATTINY85-P, P1 CONN_01X02, P2 CONN_01X02, P3 CONN_01X02, P4 CONN_01X04, Q1 TIP41C, U1 7805, U2 MCP4801, U3 LM358

Commit message: Tweaking PCB text layout
Parts:
- added G***: OSHW-logo_silkscreen-back_4mm, OSHW-logo:OSHW-logo_silkscreen-back_4mm, F.Cu at (137.2, 42.5)
- moved G*** 1.80 mm to (137.2, 42.5)
Changed lines of the file:
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@@
     (area 94.661667 28.621666 148.285001 84.408333)
     (thickness 1.6)
-    (drawings 34)
+    (drawings 42)
     (tracks 158)
     (zones 0)
-    (modules 39)
+    (modules 40)
     (nets 25)
   )
   (page A4)
   (layers
-    (0 F.Cu signal)
+    (0 F.Cu signal hide)
     (31 B.Cu signal)
     (32 B.Adhes user)
@@
   )
   (module OSHW-logo:OSHW-logo_silkscreen-front_4mm (layer F.Cu)
-    (at 135.89 41.275)
+    (at 137.16 42.545)
     (fp_text reference G*** (at 0 2.1209) (layer F.SilkS) hide
       (effects (font (size 0.18034 0.18034) (thickness 0.03556)))
@@
       (xy -1.21158 1.79578)) (layer F.SilkS) (width 0.00254))
   )
-  (gr_text "(v1)" (at 117.729 49.403 90) (layer F.SilkS)
+  (module OSHW-logo:OSHW-logo_silkscreen-back_4mm (layer F.Cu)
+    (at 137.16 42.545)
+    (fp_text reference G*** (at 0 2.1209) (layer B.SilkS) hide
+      (effects (font (size 0.18034 0.18034) (thickness 0.03556)))
+    )
+    (fp_text value OSHW-logo_silkscreen-back_4mm (at 0 -2.1209) (layer B.SilkS) hide
+      (effects (font (size 0.18034 0.18034) (thickness 0.03556)))
+    )
+    (fp_poly (pts (xy 1.21158 1.79578) (xy 1.19126 1.78562) (xy 1.143 1.75514) (xy 1.07696 1.71196)
+      (xy 0.99822 1.65862) (xy 0.91948 1.60528) (xy 0.85344 1.5621) (xy 0.80772 1.53162)
+      (xy 0.78994 1.52146) (xy 0.77978 1.524) (xy 0.74168 1.54432) (xy 0.6858 1.57226)
+      (xy 0.65532 1.5875) (xy 0.60452 1.61036) (xy 0.57912 1.61544) (xy 0.57658 1.60782)
+      (xy 0.55626 1.56972) (xy 0.52832 1.50368) (xy 0.49022 1.41732) (xy 0.44704 1.31572)
+      (xy 0.40132 1.2065) (xy 0.3556 1.09474) (xy 0.30988 0.98806) (xy 0.27178 0.89154)
+      (xy 0.23876 0.81534) (xy 0.21844 0.75946) (xy 0.21082 0.7366) (xy 0.21336 0.73152)
+      (xy 0.23876 0.70866) (xy 0.28194 0.67564) (xy 0.37846 0.5969) (xy 0.4699 0.48006)
+      (xy 0.52832 0.34798) (xy 0.5461 0.20066) (xy 0.53086 0.06604) (xy 0.47752 -0.0635)
+      (xy 0.38608 -0.18288) (xy 0.27432 -0.26924) (xy 0.14478 -0.32512) (xy 0 -0.3429)
+      (xy -0.1397 -0.32766) (xy -0.27178 -0.27432) (xy -0.39116 -0.18542) (xy -0.43942 -0.127)
+      (xy -0.508 -0.00762) (xy -0.54864 0.11938) (xy -0.55118 0.14986) (xy -0.5461 0.2921)
+      (xy -0.50546 0.42672) (xy -0.4318 0.5461) (xy -0.32766 0.64516) (xy -0.31496 0.65532)
+      (xy -0.2667 0.69088) (xy -0.23622 0.71374) (xy -0.21082 0.73406) (xy -0.38862 1.16586)
+      (xy -0.41656 1.23444) (xy -0.46736 1.35128) (xy -0.51054 1.45288) (xy -0.54356 1.53416)
+      (xy -0.56896 1.5875) (xy -0.57912 1.61036) (xy -0.57912 1.61036) (xy -0.59436 1.6129)
+      (xy -0.62738 1.6002) (xy -0.68834 1.57226) (xy -0.72898 1.55194) (xy -0.7747 1.52908)
+      (xy -0.79502 1.52146) (xy -0.8128 1.53162) (xy -0.85598 1.55956) (xy -0.91948 1.60274)
+      (xy -0.99568 1.65354) (xy -1.06934 1.70434) (xy -1.13792 1.75006) (xy -1.18618 1.78054)
+      (xy -1.21158 1.79324) (xy -1.21412 1.79324) (xy -1.23444 1.78054) (xy -1.27508 1.75006)
+      (xy -1.3335 1.69418) (xy -1.41478 1.6129) (xy -1.42748 1.6002) (xy -1.49606 1.52908)
+      (xy -1.55194 1.47066) (xy -1.59004 1.43002) (xy -1.60274 1.41224) (xy -1.60274 1.41224)
+      (xy -1.59004 1.38684) (xy -1.55956 1.33858) (xy -1.51384 1.27) (xy -1.4605 1.19126)
+      (xy -1.31826 0.98298) (xy -1.397 0.7874) (xy -1.41986 0.72898) (xy -1.45034 0.65532)
+      (xy -1.4732 0.60452) (xy -1.4859 0.58166) (xy -1.50622 0.57404) (xy -1.55956 0.56134)
+      (xy -1.6383 0.54356) (xy -1.72974 0.52832) (xy -1.81864 0.51054) (xy -1.89738 0.4953)
+      (xy -1.9558 0.48514) (xy -1.9812 0.48006) (xy -1.98628 0.47498) (xy -1.99136 0.46228)
+      (xy -1.99644 0.43688) (xy -1.99644 0.38862) (xy -1.99898 0.31242) (xy -1.99898 0.20066)
+      (xy -1.99898 0.1905) (xy -1.99644 0.08382) (xy -1.99644 0) (xy -1.9939 -0.05334)
+      (xy -1.98882 -0.07366) (xy -1.98882 -0.07366) (xy -1.96342 -0.08128) (xy -1.90754 -0.09144)
+      (xy -1.8288 -0.10922) (xy -1.73228 -0.127) (xy -1.7272 -0.127) (xy -1.63322 -0.14478)
+      (xy -1.55448 -0.16256) (xy -1.4986 -0.17526) (xy -1.47574 -0.18288) (xy -1.47066 -0.18796)
+      (xy -1.45034 -0.22606) (xy -1.4224 -0.28448) (xy -1.39192 -0.3556) (xy -1.36144 -0.42926)
+      (xy -1.3335 -0.49784) (xy -1.31572 -0.5461) (xy -1.31064 -0.56896) (xy -1.31064 -0.56896)
+      (xy -1.32588 -0.59182) (xy -1.3589 -0.64262) (xy -1.40462 -0.70866) (xy -1.4605 -0.78994)
+      (xy -1.46304 -0.79756) (xy -1.51892 -0.8763) (xy -1.5621 -0.94488) (xy -1.59258 -0.99314)
+      (xy -1.60274 -1.01346) (xy -1.60274 -1.016) (xy -1.58496 -1.03886) (xy -1.54432 -1.08458)
+      (xy -1.4859 -1.14554) (xy -1.41478 -1.21666) (xy -1.39192 -1.23698) (xy -1.31572 -1.31318)
+      (xy -1.26238 -1.36398) (xy -1.22682 -1.38938) (xy -1.21158 -1.397) (xy -1.21158 -1.39446)
+      (xy -1.18618 -1.38176) (xy -1.13538 -1.34874) (xy -1.0668 -1.30048) (xy -0.98552 -1.24714)
+      (xy -0.98044 -1.24206) (xy -0.9017 -1.18872) (xy -0.83566 -1.143) (xy -0.7874 -1.11252)
+      (xy -0.76708 -1.09982) (xy -0.762 -1.09982) (xy -0.73152 -1.10998) (xy -0.6731 -1.12776)
+      (xy -0.60452 -1.1557) (xy -0.53086 -1.18618) (xy -0.46228 -1.21412) (xy -0.41148 -1.23698)
+      (xy -0.38862 -1.24968) (xy -0.38862 -1.25222) (xy -0.37846 -1.28016) (xy -0.36576 -1.34112)
+      (xy -0.34798 -1.4224) (xy -0.3302 -1.52146) (xy -0.32766 -1.5367) (xy -0.30988 -1.63068)
+      (xy -0.29464 -1.70942) (xy -0.28194 -1.7653) (xy -0.27686 -1.78816) (xy -0.26416 -1.7907)
+      (xy -0.2159 -1.79324) (xy -0.14478 -1.79578) (xy -0.05842 -1.79578) (xy 0.03048 -1.79578)
+      (xy 0.11684 -1.79324) (xy 0.19304 -1.7907) (xy 0.24638 -1.78816) (xy 0.26924 -1.78308)
+      (xy 0.27178 -1.78054) (xy 0.2794 -1.7526) (xy 0.2921 -1.69164) (xy 0.30988 -1.61036)
+      (xy 0.32766 -1.5113) (xy 0.3302 -1.49352) (xy 0.34798 -1.39954) (xy 0.36576 -1.3208)
+      (xy 0.37592 -1.26746) (xy 0.38354 -1.24714) (xy 0.39116 -1.24206) (xy 0.42926 -1.22428)
+      (xy 0.49276 -1.19888) (xy 0.57404 -1.16586) (xy 0.75692 -1.0922) (xy 0.98044 -1.24714)
+      (xy 1.00076 -1.25984) (xy 1.08204 -1.31572) (xy 1.14808 -1.3589) (xy 1.1938 -1.38938)
+      (xy 1.21412 -1.39954) (xy 1.21412 -1.39954) (xy 1.23698 -1.37922) (xy 1.2827 -1.33858)
+      (xy 1.34366 -1.27762) (xy 1.41224 -1.20904) (xy 1.46558 -1.1557) (xy 1.52654 -1.0922)
+      (xy 1.56718 -1.05156) (xy 1.5875 -1.02362) (xy 1.59512 -1.00584) (xy 1.59258 -0.99568)
+      (xy 1.57988 -0.97282) (xy 1.54686 -0.92456) (xy 1.50114 -0.85598) (xy 1.44526 -0.77724)
+      (xy 1.39954 -0.70866) (xy 1.35128 -0.635) (xy 1.3208 -0.58166) (xy 1.3081 -0.55372)
+      (xy 1.31064 -0.54356) (xy 1.32842 -0.50038) (xy 1.35382 -0.4318) (xy 1.38684 -0.35306)
+      (xy 1.46558 -0.17526) (xy 1.58242 -0.15494) (xy 1.65354 -0.1397) (xy 1.7526 -0.12192)
+      (xy 1.84658 -0.10414) (xy 1.9939 -0.07366) (xy 1.99898 0.46482) (xy 1.97612 0.47498)
+      (xy 1.95326 0.4826) (xy 1.89992 0.49276) (xy 1.82118 0.508) (xy 1.72974 0.52578)
+      (xy 1.651 0.54102) (xy 1.57226 0.55626) (xy 1.51638 0.56642) (xy 1.49098 0.5715)
+      (xy 1.48336 0.58166) (xy 1.46304 0.61976) (xy 1.4351 0.68072) (xy 1.40462 0.75438)
+      (xy 1.37414 0.82804) (xy 1.3462 0.89916) (xy 1.32588 0.9525) (xy 1.31826 0.98044)
+      (xy 1.32842 1.00076) (xy 1.3589 1.04648) (xy 1.40208 1.11252) (xy 1.45542 1.19126)
+      (xy 1.5113 1.27) (xy 1.55448 1.33858) (xy 1.5875 1.38684) (xy 1.6002 1.40716)
+      (xy 1.59258 1.4224) (xy 1.5621 1.4605) (xy 1.50368 1.52146) (xy 1.41478 1.61036)
+      (xy 1.39954 1.62306) (xy 1.33096 1.69164) (xy 1.27 1.74498) (xy 1.22936 1.78308)
+      (xy 1.21158 1.79578)) (layer B.SilkS) (width 0.00254))
+  )
+  (gr_text "(v1)" (at 117.729 64.389 90) (layer B.SilkS)
+    (effects (font (size 0.635 0.635) (thickness 0.127)) (justify mirror))
+  )
+  (gr_text github.com/pepaslabs/prog-cc-100mA (at 119.38 57.15 90) (layer B.SilkS)
+    (effects (font (size 0.635 0.635) (thickness 0.127)) (justify mirror))
+  )
+  (gr_text "0-100mA Programmable\nCurrent Source" (at 116.84 57.15 90) (layer B.SilkS)
+    (effects (font (size 1.016 1.016) (thickness 0.2032)) (justify mirror))
+  )
+  (gr_text GND (at 102.235 53.34) (layer B.SilkS)
+    (effects (font (size 0.635 0.635) (thickness 0.127)) (justify mirror))
+  )
+  (gr_text RX (at 102.235 50.8) (layer B.SilkS)
+    (effects (font (size 0.635 0.635) (thickness 0.127)) (justify mirror))
+  )
+  (gr_text TX (at 102.235 48.26) (layer B.SilkS)
+    (effects (font (size 0.635 0.635) (thickness 0.127)) (justify mirror))
+  )
+  (gr_text 5V (at 102.235 45.72) (layer B.SilkS)
+    (effects (font (size 0.635 0.635) (thickness 0.127)) (justify mirror))
+  )
+  (gr_text "TTL\nSERIAL" (at 99.695 42.545) (layer B.SilkS)
+    (effects (font (size 0.635 0.635) (thickness 0.127)) (justify mirror))
+  )
+  (gr_text "(v1)" (at 117.729 49.911 90) (layer F.SilkS)
     (effects (font (size 0.635 0.635) (thickness 0.127)))
   )
@@
     (effects (font (size 0.762 0.762) (thickness 0.1524)))
   )
-  (gr_text github.com/pepaslabs/prog-cc-100mA (at 119.38 57.785 90) (layer F.SilkS)
+  (gr_text github.com/pepaslabs/prog-cc-100mA (at 119.38 57.15 90) (layer F.SilkS)
     (effects (font (size 0.635 0.635) (thickness 0.127)))
   )
-  (gr_text "0-100mA Programmable\nCurrent Source" (at 116.84 56.515 90) (layer F.SilkS)
+  (gr_text "0-100mA Programmable\nCurrent Source" (at 116.84 57.15 90) (layer F.SilkS)
     (effects (font (size 1.016 1.016) (thickness 0.2032)))
   )
