File: kicad/prog-cc-100mA.sch (KiCad schematic (older format))
At the start: 34 parts, among them IC1 ATTINY85-P, P1 CONN_01X02, P2 CONN_01X02, P3 CONN_01X02, P4 CONN_01X04, Q1 TIP41C, U1 7805, U2 MCP4801, U3 LM358

Commit message: Tweaking a few part designations
Parts:
- removed P1, P2, P3: CONN_01X02, Pin_Headers:Pin_Header_Straight_1x02, symbol CONN_01X02
- removed P4: CONN_01X04, Pin_Headers:Pin_Header_Straight_1x04, symbol CONN_01X04
- removed R5: 220, PL_resistors:R_AXIAL_0W25_059A_PL, symbol R_0W25_1PCT
- added P1, P2, P3: CONN_2X1, symbol CONN_2X1
- added P4: CONN_4X1, symbol CONN_4X1
- added R5: 220, symbol R_0W25
- C4, C5: value 100uF -> 10uF
- D1, D2: value 1N4001 -> 1N4148
Changed lines of the file:
@@
 LIBS:valves
 LIBS:prog-cc-100mA-cache
-EELAYER 25 0
+EELAYER 27 0
 EELAYER END
 $Descr USLedger 17000 11000
@@
 Sheet 1 1
 Title ""
-Date ""
+Date "10 may 2017"
 Rev ""
 Comp ""
@@
 L GND #PWR01
 U 1 1 58ED2344
-P 12100 8150
-F 0 "#PWR01" H 12100 7900 50  0001 C CNN
-F 1 "GND" H 12100 8000 50  0001 C CNN
-F 2 "" H 12100 8150 50  0000 C CNN
-F 3 "" H 12100 8150 50  0000 C CNN
-	1    12100 8150
+P 12100 8200
+F 0 "#PWR01" H 12100 7950 50  0001 C CNN
+F 1 "GND" H 12100 8050 50  0001 C CNN
+F 2 "" H 12100 8200 50  0000 C CNN
+F 3 "" H 12100 8200 50  0000 C CNN
+	1    12100 8200
 	1    0    0    -1
 $EndComp
@@
 Text Notes 10600 5000 0    60   ~ 0
 Difference amp, 1x gain
-$Comp
-L R_0W25_1PCT R5
-U 1 1 58EFCA7C
-P 11300 4500
-F 0 "R5" V 11380 4500 40  0000 C CNN
-F 1 "220" V 11300 4500 40  0000 C CNN
-F 2 "PL_resistors:R_AXIAL_0W25_059A_PL" V 11230 4500 30  0001 C CNN
-F 3 "" H 11300 4500 30  0000 C CNN
-	1    11300 4500
-	0    1    1    0
-$EndComp
 $Comp
 L 7805 U1
@@
 Text GLabel 8300 5500 1    60   Input ~ 0
 SDO
-$Comp
-L CONN_01X02 P1
-U 1 1 58F6DF60
-P 12400 1800
-F 0 "P1" H 12400 1950 50  0000 C CNN
-F 1 "CONN_01X02" V 12500 1800 50  0000 C CNN
-F 2 "Pin_Headers:Pin_Header_Straight_1x02" H 12400 1800 50  0001 C CNN
-F 3 "" H 12400 1800 50  0000 C CNN
-	1    12400 1800
-	1    0    0    -1
-$EndComp
-$Comp
-L CONN_01X02 P3
-U 1 1 58F6F564
-P 12400 8000
-F 0 "P3" H 12400 8150 50  0000 C CNN
-F 1 "CONN_01X02" V 12500 8000 50  0000 C CNN
-F 2 "Pin_Headers:Pin_Header_Straight_1x02" H 12400 8000 50  0001 C CNN
-F 3 "" H 12400 8000 50  0000 C CNN
-	1    12400 8000
-	1    0    0    -1
-$EndComp
 Text GLabel 11600 1500 1    60   Input ~ 0
 +V
@@
 P 11600 1800
 F 0 "C4" H 11620 1860 30  0000 L BNN
-F 1 "100uF" H 11620 1710 30  0000 L TNN
+F 1 "10uF" H 11620 1710 30  0000 L TNN
 F 2 "PL_capacitors:ELCAP_10_20_V_059A" H 11638 1650 30  0001 C CNN
 F 3 "" H 11600 1800 60  0000 C CNN
@@
 P 11900 1600
 F 0 "D1" H 11900 1700 40  0000 C CNN
-F 1 "1N4001" H 11900 1500 40  0000 C CNN
+F 1 "1N4148" H 11900 1500 40  0000 C CNN
 F 2 "PL_diodes:DIODE_1A_069A_PL" H 11900 1600 60  0001 C CNN
 F 3 "" H 11900 1600 60  0000 C CNN
@@
 $EndComp
 $Comp
-L CONN_01X02 P2
-U 1 1 58F876AE
-P 12400 2400
-F 0 "P2" H 12400 2550 50  0000 C CNN
-F 1 "CONN_01X02" V 12500 2400 50  0000 C CNN
-F 2 "Pin_Headers:Pin_Header_Straight_1x02" H 12400 2400 50  0001 C CNN
-F 3 "" H 12400 2400 50  0000 C CNN
-	1    12400 2400
-	1    0    0    -1
-$EndComp
-$Comp
 L C_EL C5
 U 1 1 58F876B4
 P 11600 2400
 F 0 "C5" H 11620 2460 30  0000 L BNN
-F 1 "100uF" H 11620 2310 30  0000 L TNN
+F 1 "10uF" H 11620 2310 30  0000 L TNN
 F 2 "PL_capacitors:ELCAP_10_20_V_059A" H 11638 2250 30  0001 C CNN
 F 3 "" H 11600 2400 60  0000 C CNN
@@
 P 11900 2600
 F 0 "D2" H 11900 2700 40  0000 C CNN
-F 1 "1N4001" H 11900 2500 40  0000 C CNN
+F 1 "1N4148" H 11900 2500 40  0000 C CNN
 F 2 "PL_diodes:DIODE_1A_069A_PL" H 11900 2600 60  0001 C CNN
 F 3 "" H 11900 2600 60  0000 C CNN
@@
 Text Notes 7250 1850 0    100  ~ 0
 0-100mA Programmable Current Source
-$Comp
-L CONN_01X04 P4
-U 1 1 58F8F01B
-P 8700 7500
-F 0 "P4" H 8700 7750 50  0000 C CNN
-F 1 "CONN_01X04" V 8800 7500 50  0000 C CNN
-F 2 "Pin_Headers:Pin_Header_Straight_1x04" H 8700 7500 50  0001 C CNN
-F 3 "" H 8700 7500 50  0000 C CNN
-	1    8700 7500
-	1    0    0    -1
-$EndComp
 Text GLabel 8400 7250 1    60   Input ~ 0
 +5V
@@
 	12100 4700 12100 5750
 Wire Wire Line
-	12100 6650 12100 7950
+	12100 6650 12100 8000
 Wire Wire Line
 	11800 4500 11500 4500
@@
 	8050 5800 8450 5800
 Wire Wire Line
-	12200 8050 12100 8050
-Wire Wire Line
-	12100 8050 12100 8150
-Wire Wire Line
 	11150 7550 11000 7550
 Wire Wire Line
@@
 Connection ~ 9400 4400
 Wire Wire Line
-	12100 7950 12200 7950
-Wire Wire Line
 	11600 1500 11600 1650
 Wire Wire Line
@@
 	12100 1600 12200 1600
 Wire Wire Line
-	12200 1600 12200 1750
-Wire Wire Line
-	12200 1850 12200 2000
-Wire Wire Line
 	11600 1950 11600 2250
 Wire Wire Line
 	11600 2200 12200 2200
 Connection ~ 11600 2200
-Wire Wire Line
-	12200 2200 12200 2350
-Wire Wire Line
-	12200 2450 12200 2600
 Connection ~ 11600 2600
 Wire Wire Line
@@
 Wire Wire Line
 	12200 2600 12100 2600
-Text Notes 12650 8000 0    60   ~ 0
+Text Notes 12700 8100 0    60   ~ 0
 Output
-Text Notes 12650 1800 0    60   ~ 0
+Text Notes 12750 1850 0    60   ~ 0
 Positive supply
-Text Notes 12650 2400 0    60   ~ 0
+Text Notes 12750 2400 0    60   ~ 0
 Negative supply
+Wire Wire Line
+	12200 1600 12200 1750
+Wire Wire Line
+	12200 1850 12200 2000
+Wire Wire Line
+	12200 2200 12200 2350
+Wire Wire Line
+	12200 2450 12200 2600
+$Comp
+L CONN_2X1 P3
+U 1 1 5913A735
+P 12400 8050
+F 0 "P3" V 12400 8050 40  0000 C CNN
+F 1 "CONN_2X1" V 12500 8050 40  0000 C CNN
+F 2 "" H 12450 8050 60  0000 C CNN
+F 3 "" H 12450 8050 60  0000 C CNN
+	1    12400 8050
+	1    0    0    -1
+$EndComp
+Wire Wire Line
+	12100 8000 12200 8000
+Wire Wire Line
+	12200 8100 12100 8100
+Wire Wire Line
+	12100 8100 12100 8200
+$Comp
+L CONN_2X1 P2
+U 1 1 5913A850
+P 12400 2400
+F 0 "P2" V 12400 2400 40  0000 C CNN
+F 1 "CONN_2X1" V 12500 2400 40  0000 C CNN
+F 2 "" H 12450 2400 60  0000 C CNN
+F 3 "" H 12450 2400 60  0000 C CNN
+	1    12400 2400
+	1    0    0    -1
+$EndComp
+$Comp
+L CONN_2X1 P1
+U 1 1 5913A856
+P 12400 1800
+F 0 "P1" V 12400 1800 40  0000 C CNN
+F 1 "CONN_2X1" V 12500 1800 40  0000 C CNN
+F 2 "" H 12450 1800 60  0000 C CNN
+F 3 "" H 12450 1800 60  0000 C CNN
+	1    12400 1800
+	1    0    0    -1
+$EndComp
+$Comp
+L CONN_4X1 P4
+U 1 1 5913AA84
+P 8700 7500
+F 0 "P4" V 8700 7500 40  0000 C CNN
+F 1 "CONN_4X1" V 8800 7500 40  0000 C CNN
+F 2 "" H 8750 7600 60  0000 C CNN
+F 3 "" H 8750 7600 60  0000 C CNN
+	1    8700 7500
+	1    0    0    -1
+$EndComp
+$Comp
+L R_0W25 R5
+U 1 1 5913ABB7
+P 11300 4500
+F 0 "R5" V 11380 4500 40  0000 C CNN
+F 1 "220" V 11300 4500 40  0000 C CNN
+F 2 "" V 11230 4500 30  0000 C CNN
+F 3 "" H 11300 4500 30  0000 C CNN
+	1    11300 4500
+	0    1    1    0
+$EndComp
 $EndSCHEMATC
